Commit message: update config and urdf

File: unitree_d1_description/urdf/ros2_control/unitree_d1_ros2_control.xacro (robot description, xacro)
@@ -1,5 +1,5 @@
 <?xml version="1.0"?>
 <robot xmlns:xacro="http://ros.org/wiki/xacro">
-  <xacro:macro name="unitree_d1_ros2_control" params="prefix sim_gazebo" >
+  <xacro:macro name="unitree_d1_ros2_control" params="prefix sim_gazebo gripper:=d1_2f" >
     <ros2_control name="ArmHardwareInterface" type="system">
         <xacro:if value="${sim_gazebo}">
@@ -12,8 +12,8 @@
                 <plugin>d1_hardware_interface/D1HardwareInterface</plugin>
                 <!-- <param name="topic_sufix">asda</param> -->
-                <!-- <xacro:if value="${gripper == 'z1_1f'}">
-                    <param name="gripper">true</param>
-                </xacro:if>
-                <xacro:unless value="${gripper == 'z1_1f'}">
+                <!-- <xacro:if value="${gripper == 'd1_2f'}"> -->
+                <param name="gripper">${gripper}</param>
+                <!-- </xacro:if> -->
+                <!-- <xacro:unless value="${gripper == 'z1_1f'}">
                     <param name="gripper">false</param>
                 </xacro:unless> -->
@@ -116,4 +116,12 @@
             <state_interface name="effort"/> -->
         </joint>
+        <!-- Default Gripper -->
+        <xacro:if value="${gripper == 'd1_2f' and not sim_gazebo}">
+            <joint name="${prefix}joint_L">
+                <command_interface name="position" />
+                <state_interface name="position" />
+                <state_interface name="velocity" />
+            </joint>
+        </xacro:if>
     </ros2_control>
   </xacro:macro>

File: unitree_d1_description/urdf/unitree_d1.urdf.xacro (robot description, xacro)
@@ -29,3 +29,5 @@
         </xacro:load_gripper>
     </xacro:unless>
+    <xacro:include filename="$(find unitree_d1_description)/urdf/ros2_control/unitree_d1_ros2_control.xacro" />
+    <xacro:unitree_d1_ros2_control prefix="$(arg prefix)" sim_gazebo="$(arg sim_gazebo)" gripper="$(arg gripper)"/>
 </robot>

File: unitree_d1_description/urdf/unitree_d1_macro.urdf.xacro (robot description, xacro)
@@ -217,6 +217,4 @@
             <xacro:unitree_d1_gazebo parent="${parent}" prefix="${prefix}" use_camera="${use_camera}" />
         </xacro:if>
-        <xacro:include filename="$(find unitree_d1_description)/urdf/ros2_control/unitree_d1_ros2_control.xacro" />
-        <xacro:unitree_d1_ros2_control prefix="${prefix}" sim_gazebo="${sim_gazebo}" />
     </xacro:macro>
 </robot>
