Commit message: test new d1

File: unitree_d1_description/urdf/gz/unitree_d1.gazebo.xacro (robot description, xacro)
@@ -1,5 +1,5 @@
 <?xml version="1.0"?>
 <robot xmlns:xacro="http://ros.org/wiki/xacro">
-  <xacro:macro name="unitree_d1_gazebo" params="parent prefix use_camera">
+  <xacro:macro name="unitree_d1_gazebo" params="parent prefix use_camera namespace">
     <gazebo reference="${prefix}base_link">
         <material>Gazebo/Dark_Grey</material>
@@ -51,4 +51,7 @@
         <plugin filename="gz_ros2_control-system" name="gz_ros2_control::GazeboSimROS2ControlPlugin">
           <parameters>$(find arms_bringup)/config/ros2_control.yaml</parameters>
+            <ros>
+                <namespace>${namespace}</namespace>
+            </ros>
         </plugin>
       </gazebo>

File: unitree_d1_description/urdf/ros2_control/unitree_d1_ros2_control.xacro (robot description, xacro)
@@ -33,6 +33,5 @@
                 <state_interface name="position" />
             </xacro:unless>
-            <!-- <state_interface name="velocity"/>
-            <state_interface name="effort"/> -->
+            <state_interface name="velocity" />
         </joint>
         <joint name="${prefix}joint_2">
@@ -49,6 +48,5 @@
                 <state_interface name="position" />
             </xacro:unless>
-            <!-- <state_interface name="velocity"/>
-            <state_interface name="effort"/> -->
+            <state_interface name="velocity" />
         </joint>
         <joint name="${prefix}joint_3">
@@ -65,6 +63,5 @@
                 <state_interface name="position" />
             </xacro:unless>
-            <!-- <state_interface name="velocity"/>
-            <state_interface name="effort"/> -->
+            <state_interface name="velocity" />
         </joint>
         <joint name="${prefix}joint_4">
@@ -81,6 +78,5 @@
                 <state_interface name="position" />
             </xacro:unless>
-            <!-- <state_interface name="velocity"/>
-            <state_interface name="effort"/> -->
+            <state_interface name="velocity" />
         </joint>
         <joint name="${prefix}joint_5">
@@ -97,6 +93,5 @@
                 <state_interface name="position" />
             </xacro:unless>
-            <!-- <state_interface name="velocity"/>
-            <state_interface name="effort"/> -->
+            <state_interface name="velocity" />
         </joint>
         <joint name="${prefix}joint_6">
@@ -113,6 +108,5 @@
                 <state_interface name="position" />
             </xacro:unless>
-            <!-- <state_interface name="velocity"/>
-            <state_interface name="effort"/> -->
+            <state_interface name="velocity" />
         </joint>
         <!-- Default Gripper -->

File: unitree_d1_description/urdf/unitree_d1.urdf.xacro (robot description, xacro)
@@ -6,5 +6,8 @@
     <xacro:arg name="use_camera" default="false" />
     <xacro:arg name="prefix" default=""/>
+    <xacro:arg name="namespace" default="" />
     <xacro:arg name="gripper" default="" />
+    <xacro:arg name="gripper_xyz" default="0.0 0.0 0.0" />
+    <xacro:arg name="gripper_rpy" default="0.0 0.0 0.0" />
     <xacro:include filename="$(find unitree_d1_description)/urdf/camera/_materials.urdf.xacro" />
     <xacro:include filename="$(find unitree_d1_description)/urdf/unitree_d1_macro.urdf.xacro" />
@@ -13,4 +16,5 @@
             parent="world"
             prefix="$(arg prefix)"
+            namespace="$(arg namespace)"
             sim_gazebo="$(arg sim_gazebo)"
             gripper="$(arg gripper)"
@@ -26,5 +30,5 @@
             sim_gazebo="$(arg sim_gazebo)">
             <!-- <origin rpy="-1.5714 -1.5708 0" xyz="-0.0056012 -0.029636 0.0706" /> -->
-            <origin rpy="0 0 0" xyz="0 0 0" />
+            <origin rpy="$(arg gripper_rpy)" xyz="$(arg gripper_xyz)" />
         </xacro:load_gripper>
     </xacro:unless>

File: unitree_d1_description/urdf/unitree_d1_macro.urdf.xacro (robot description, xacro)
@@ -4,5 +4,5 @@
     <!-- Propagate last link name information because it is the gripper's parent link -->
     <xacro:property name="last_arm_link" value="Link6" />
-    <xacro:macro name="load_arm" params="*origin parent prefix sim_gazebo gripper use_camera">
+    <xacro:macro name="load_arm" params="*origin parent prefix sim_gazebo gripper use_camera namespace">
         <joint name="${prefix}base_joint" type="fixed">
             <xacro:insert_block name="origin" />
@@ -215,5 +215,5 @@
         <xacro:if value="${sim_gazebo}">
             <xacro:include filename="$(find unitree_d1_description)/urdf/gz/unitree_d1.gazebo.xacro" />
-            <xacro:unitree_d1_gazebo parent="${parent}" prefix="${prefix}" use_camera="${use_camera}" />
+            <xacro:unitree_d1_gazebo parent="${parent}" prefix="${prefix}" use_camera="${use_camera}" namespace="${namespace}" />
         </xacro:if>
     </xacro:macro>
